File: hw/RocSync_testing.kicad_pcb (KiCad board)
At the start: 2 copper layers, 250 x 250 mm, 310 parts, among them J1 USB_C_Receptacle_PowerOnly_6P, J2 BATT, J3 PROG, SW1 ON/OFF, SW2 RESET, SW3 MODE, U1 BQ24075RGT, U10 TLC59283, U11 BCR420UW6Q, U12 BCR420UW6Q, U13 BCR420UW6Q, U14 BCR420UW6Q, U2 CH32V003FxUx, U3 TLC59283, U4 TLC59283, U5 TLC59283, U6 TLC59283, U7 TLC59283, U8 TLC59283, U9 TLC59283, Y1 Crystal_GND24

Commit message: [hw] rev 2
Parts:
- removed C15: 0.1uf, Capacitor_SMD:C_0402_1005Metric
- removed the C5 at (106.7, 27.6)
- removed the G*** at (125.0, 219.8)
- removed JP1: CHG BOOST, Jumper:SolderJumper-2_P1.3mm_Open_RoundedPad1.0x1.5mm
- removed R14: 2.7k, Resistor_SMD:R_0603_1608Metric
- removed U10: TLC59283, Package_DFN_QFN:Texas_RGE0024C_VQFN-24-1EP_4x4mm_P0.5mm_EP2.1x2.1mm_ThermalVias
- added C16: 1uf, Capacitor_SMD:C_0402_1005Metric, F.Cu at (46.8, 94.8)
- added C17: 10nF, Capacitor_SMD:C_0402_1005Metric, F.Cu at (43.4, 92.0)
- added C19: 0.1uf, Capacitor_SMD:C_0402_1005Metric, F.Cu at (205.5, 103.0)
- added C29: 0.1uf, Capacitor_SMD:C_0402_1005Metric, F.Cu at (149.5, 32.0)
- added C7: 1uf, Capacitor_SMD:C_0402_1005Metric, F.Cu at (49.9, 94.4)
- added D233: IR LED, custom_footprints:XYC-HIR76C-LX4, F.Cu at (95.0, 59.0)
- added D234: IR LED, custom_footprints:XYC-HIR76C-LX4, F.Cu at (107.0, 59.0)
- added D235: IR LED, custom_footprints:XYC-HIR76C-LX4, F.Cu at (119.0, 59.0)
- added D236: IR LED, custom_footprints:XYC-HIR76C-LX4, F.Cu at (131.0, 59.0)
- added D237: IR LED, custom_footprints:XYC-HIR76C-LX4, F.Cu at (143.0, 59.0)
- added D238: IR LED, custom_footprints:XYC-HIR76C-LX4, F.Cu at (155.0, 59.0)
- added D239: IR LED, custom_footprints:XYC-HIR76C-LX4, F.Cu at (167.0, 59.0)
- added D240: IR LED, custom_footprints:XYC-HIR76C-LX4, F.Cu at (179.0, 59.0)
- added D273: IR LED, custom_footprints:XYC-HIR76C-LX4, F.Cu at (5.00, 5.00)
- added D274: LED, custom_footprints:HL-A-3528, F.Cu at (5.00, 20.0)
- added J4: Conn_01x04_Socket, Connector_PinHeader_2.54mm:PinHeader_1x04_P2.54mm_Vertical, B.Cu at (128.8, 21.0)
- added R21: 5.1k, Resistor_SMD:R_0402_1005Metric, F.Cu at (205.5, 98.0)
- added R22: 1.8k, Resistor_SMD:R_0402_1005Metric, F.Cu at (205.5, 99.0)
- added R24: 510, Resistor_SMD:R_0402_1005Metric, F.Cu at (205.5, 101.0)
- added R25: 100, Resistor_SMD:R_0402_1005Metric, F.Cu at (47.0, 68.0)
- added R26: 10k, Resistor_SMD:R_0402_1005Metric, F.Cu at (39.4, 94.0)
- added R27: 2k, Resistor_SMD:R_0402_1005Metric, F.Cu at (205.5, 102.0)
- added R32: 2.7k, Resistor_SMD:R_0402_1005Metric, F.Cu at (102.5, 27.0)
- added R38: 2.7k, Resistor_SMD:R_0402_1005Metric, F.Cu at (149.8, 30.2)
- added SW4: SW_Push, custom_footprints:SW_Push_1P1T_NO_6x6mm_H9.5mm, B.Cu at (187.0, 119.2)
- added SW5: SW_Push, custom_footprints:SW_Push_1P1T_NO_6x6mm_H9.5mm, B.Cu at (187.0, 129.2)
- added SW6: SW_Push, custom_footprints:SW_Push_1P1T_NO_6x6mm_H9.5mm, B.Cu at (177.0, 119.2)
- added SW7: SW_Push, custom_footprints:SW_Push_1P1T_NO_6x6mm_H9.5mm, B.Cu at (197.0, 119.2)
- added U15: BCR420UW6Q, Package_TO_SOT_SMD:SOT-23-6, F.Cu at (44.0, 69.0)
- added U16: TPS7A2025, Package_TO_SOT_SMD:SOT-23-5, F.Cu at (47.9, 91.9)
- added U18: TLC59283, Package_DFN_QFN:Texas_RGE0024C_VQFN-24-1EP_4x4mm_P0.5mm_EP2.1x2.1mm_ThermalVias, F.Cu at (101.0, 31.0)
- added U26: TLC59283, Package_DFN_QFN:Texas_RGE0024C_VQFN-24-1EP_4x4mm_P0.5mm_EP2.1x2.1mm_ThermalVias, F.Cu at (153.0, 34.0)
- C18: value 0.1uf -> 10pF
- C6: value 10pf -> 0.1uf
- D211, D212, D213, D214, D215, D216: value LED -> IR LED; footprint custom_footprints:HL-A-3528 -> custom_footprints:XYC-HIR76C-LX4
- D221, D222, D223, D224, D225, D226, D227, D228, D229, D230: value IR LED -> LED; footprint custom_footprints:XYC-HIR76C-LX4 -> custom_footprints:HL-A-3528
- G***: value LOGO -> aruco_4x4_1000-21; footprint LOGO -> custom_footprints:aruco_4x4_1000-21
- G***: footprint custom_footprints:orx -> custom_footprints:orx_logo
- J3: value PROG -> Conn_01x03_Pin
- R10, R11, R12, R13, R7, R8, R9: footprint Resistor_SMD:R_0603_1608Metric -> Resistor_SMD:R_0402_1005Metric
- R23: value 1.18k -> 820
- R3: renamed from R22; value 1.18k -> 1.1k
- R4: renamed from R3; value 2k -> 590
- SW2: footprint Button_Switch_SMD:SW_Push_1P1T_NO_6x6mm_H9.5mm -> custom_footprints:SW_Push_1P1T_NO_6x6mm_H9.5mm
- SW3: value MODE -> SW_Push; footprint Button_Switch_SMD:SW_Push_1P1T_NO_6x6mm_H9.5mm -> custom_footprints:SW_Push_1P1T_NO_6x6mm_H9.5mm
- Y1: value Crystal_GND24 -> huaxindianzi 2T024000VX; footprint Crystal:Crystal_SMD_2520-4Pin_2.5x2.0mm -> Oscillator:Oscillator_SMD_SeikoEpson_TG2520SMN-xxx-xxxxxx-4Pin_2.5x2.0mm
- moved R23 156.3 mm to (205.5, 100.0), turned to 0 degrees
- moved J3 111.5 mm to (49.0, 109.2)
- moved D231 106.6 mm to (71.0, 59.0)
- moved D232 102.6 mm to (83.0, 59.0)
- moved C4 95.8 mm to (37.0, 95.5)
- moved C5 95.6 mm to (42.8, 95.4)
- moved U2 95.1 mm to (39.9, 97.4)
- moved R20 95.1 mm to (38.0, 100.2)
- moved Y1 93.6 mm to (40.9, 91.7), turned to -90 degrees
- moved D220 90.0 mm to (179.0, 47.0)
- moved C18 88.4 mm to (41.4, 94.0), turned to 0 degrees
- moved D219 86.0 mm to (167.0, 47.0)
- moved D218 82.0 mm to (155.0, 47.0)
- moved D217 78.0 mm to (143.0, 47.0)
- moved D211 74.2 mm to (71.0, 47.0)
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- renumbered C3 to C2, C2 to C3, C7 to C5, D233 to D265, D237 to D266, D234 to D267, D238 to D268, D235 to D269, D239 to D270, D236 to D271, D240 to D272, D241 to D275, D242 to D276, D243 to D277, R6 to R19, R19 to R20, R4 to R5, R5 to R6
Connections:
- C18 pad 1: Net-(U2-PC2) -> /OSCI
- C6 pad 1: /OSCI -> GND
- C6 pad 2: GND -> VCC
- D211 pad 2: VCC -> Net-(D201-K)
- D212 pad 2: VCC -> Net-(D202-K)
- D213 pad 2: VCC -> Net-(D203-K)
- D214 pad 2: VCC -> Net-(D204-K)
- D215 pad 2: VCC -> Net-(D205-K)
- D216 pad 2: VCC -> Net-(D206-K)
- D217 pad 2: Net-(D201-K) -> Net-(D207-K)
- D218 pad 2: Net-(D202-K) -> Net-(D208-K)
- D219 pad 2: Net-(D203-K) -> Net-(D209-K)
- D220 pad 2: Net-(D204-K) -> Net-(D210-K)
- D221 pad 2: Net-(D205-K) -> VCC
- D222 pad 2: Net-(D206-K) -> VCC
- D223 pad 2: Net-(D207-K) -> VCC
- D224 pad 2: Net-(D208-K) -> VCC
- D225 pad 2: Net-(D209-K) -> VCC
- D226 pad 2: Net-(D210-K) -> VCC
- D227 pad 2: Net-(D211-K) -> VCC
- D228 pad 2: Net-(D212-K) -> VCC
- D229 pad 2: Net-(D213-K) -> VCC
- D230 pad 2: Net-(D214-K) -> VCC
- D231 pad 2: Net-(D215-K) -> Net-(D221-K)
- D232 pad 2: Net-(D216-K) -> Net-(D222-K)
- J2 pad 1: GND -> +BATT
- J2 pad 2: +BATT -> GND
- R23 pad 2: Net-(U1-ISET) -> Net-(R23-Pad2)
- SW3 pad 1: GND -> Net-(R21-Pad1)
- SW3 pad 2: Net-(U2-PC2) -> GND
- U2 pad 11: unconnected-(U2-PC4-Pad11) -> /RING_LATCH
- U2 pad 3: /OSCO -> /BTN_LADDER
- U2 pad 8: /RING_LATCH -> /SDA
- U2 pad 9: Net-(U2-PC2) -> /SCL
- Y1 pad 1: /OSCI -> unconnected-(Y1-NC/GND-Pad1)
- Y1 pad 3: /OSCO -> /OSCI
- Y1 pad 4: GND -> Net-(U16-VOUT)
Routing:
- net /BTN_LADDER: track 0.00 -> 203.5 mm, vias 0 -> 4
- net /COUNTER_LATCH: track 19.8 -> 170.1 mm, vias 2 -> 4
- net /COUNTER_BLANK: track 20.6 -> 169.6 mm, vias 2 -> 4
- net /SCL: track 0.00 -> 139.0 mm, vias 0 -> 3
- net /SDA: track 0.00 -> 138.1 mm, vias 0 -> 3
- net VCC: track 695.9 -> 825.0 mm, vias 23 -> 30
- net Net-(U2-PC2): track 121.6 -> 0.00 mm, vias 1 -> 0
- net /COUNTER_DATA: track 17.5 -> 107.7 mm, vias 2 -> 4
- net /RING_BLANK: track 543.7 -> 615.1 mm, vias 12 -> 18
- net Net-(D274-K): track 0.00 -> 70.0 mm, vias 0 -> 2
- net /CLK: track 539.8 -> 607.5 mm, vias 12 -> 16
- net /RING_DATA: track 36.1 -> 93.4 mm, vias 2 -> 4
- net Net-(U18-SOUT): track 0.00 -> 51.3 mm
- net Net-(D220-K): track 35.8 -> 86.4 mm, vias 0 -> 2
- net /CORNER_PWM: track 521.4 -> 472.2 mm
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Other:
- board text added: "GND"
- board text added: "OLED"
- board text added: "Rev2"
- board text added: "SWDIO"
- board text added: "VCC"
