File: hw/corner.kicad_sch (KiCad schematic)
At the start: 16 parts, among them U11 BCR420UW6Q, U12 BCR420UW6Q, U13 BCR420UW6Q, U14 BCR420UW6Q

Commit message: [hw] rev 2
Parts:
- added D273: IR LED, custom_footprints:XYC-HIR76C-LX4, symbol Device:LED
- added D274: LED, custom_footprints:HL-A-3528, symbol Device:LED
- added R25: 100, Resistor_SMD:R_0402_1005Metric, symbol Device:R
- added U15: BCR420UW6Q, Package_TO_SOT_SMD:SOT-23-6, symbol custom_symbols:BCR420UW6Q
- renumbered D233 to D265, D237 to D266, D234 to D267, D238 to D268, D235 to D269, D239 to D270, D236 to D271, D240 to D272
Connections:
- net EN: now also U15.1 (EN)
- net GND: now also R25.2, U15.4 (GND)
- net VCC: now also D273.2 (A)
- new net: D274.1 (K), U15.2 (OUT)
- new net: R25.1, U15.6 (R_EXT)
- new net: D273.1 (K), D274.2 (A)
