File: hw/counter.kicad_sch (KiCad schematic)
At the start: 35 parts, among them U8 TLC59283

Commit message: [hw] rev 2
Parts:
- added C29: 0.1uf, Capacitor_SMD:C_0402_1005Metric, symbol Device:C
- added D227, D228, D229, D230: LED, custom_footprints:HL-A-3528, symbol Device:LED
- added D237, D238, D239, D240: IR LED, custom_footprints:XYC-HIR76C-LX4, symbol Device:LED
- added R38: 2.7k, Resistor_SMD:R_0402_1005Metric, symbol Device:R
- added U26: TLC59283, Package_DFN_QFN:Texas_RGE0024C_VQFN-24-1EP_4x4mm_P0.5mm_EP2.1x2.1mm_ThermalVias, symbol custom_symbols:TLC59283
- R32: renamed from R12; footprint Resistor_SMD:R_0603_1608Metric -> Resistor_SMD:R_0402_1005Metric
- renumbered C13 to C6, D81 to D201, D82 to D202, D83 to D203, D84 to D204, D85 to D205, D86 to D206, D87 to D207, D88 to D208, D89 to D209, D90 to D210, D181 to D211, D182 to D212, D183 to D213, D184 to D214, D185 to D215, D186 to D216, D187 to D217, D188 to D218, D189 to D219, D190 to D220, D91 to D221, D92 to D222, D93 to D223, D94 to D224, D95 to D225, D96 to D226, D191 to D231, D192 to D232, D193 to D233, D194 to D234, D195 to D235, D196 to D236, U8 to U18
Connections:
- net BLANK: now also U26.18 (BLANK)
- net CLK: now also U26.24 (SCLK)
- net DOUT: now also U26.19 (SOUT); no longer U18.19 (SOUT)
- net GND: now also C29.1, R38.1, U26.22 (GND), U26.25 (PowerPAD)
- net LAT: now also U26.1 (LAT)
- net VCC: now also C29.2, D227.2 (A), D228.2 (A), D229.2 (A), D230.2 (A), U26.21 (VCC)
- new net: U18.19 (SOUT), U26.23 (SIN)
- new net: D227.1 (K), D237.2 (A)
- new net: D238.1 (K), U26.3 (OUT1)
- new net: D228.1 (K), D238.2 (A)
- new net: D230.1 (K), D240.2 (A)
- new net: D229.1 (K), D239.2 (A)
- new net: D237.1 (K), U26.2 (OUT0)
- new net: R38.2, U26.20 (IREF)
- new net: D239.1 (K), U26.4 (OUT2)
- new net: D240.1 (K), U26.5 (OUT3)
Other:
- moved on the sheet: C6
