File: hw/ring_segment_small.kicad_sch (KiCad schematic)
At the start: 11 parts, among them U9 TLC59283

Commit message: [hw] rev 2
Parts:
- R13: footprint Resistor_SMD:R_0603_1608Metric -> Resistor_SMD:R_0402_1005Metric
Changed lines of the file:
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@@
 (kicad_sch
-	(version 20231120)
+	(version 20250114)
 	(generator "eeschema")
-	(generator_version "8.0")
+	(generator_version "9.0")
 	(paper "A4")
+	(text "R_IREF configured for 20 mA sink current"
+		(exclude_from_sim no)
+		(at 56.642 106.172 0)
+		(effects
+			(font
+				(size 1.27 1.27)
+				(color 249 0 0 1)
+			)
+		)
+	)
 	(junction
 		(at 118.11 33.02)
@@
 		)
 	)
-	(text "R_IREF configured for 20 mA sink current"
-		(exclude_from_sim no)
-		(at 56.642 106.172 0)
-		(effects
-			(font
-				(size 1.27 1.27)
-				(color 249 0 0 1)
-			)
-		)
-	)
 	(hierarchical_label "CLK"
 		(shape input)
 		(at 53.34 78.74 180)
-		(fields_autoplaced yes)
 		(effects
 			(font
@@
 		(shape input)
 		(at 53.34 76.2 180)
-		(fields_autoplaced yes)
 		(effects
 			(font
@@
 		(shape input)
 		(at 53.34 73.66 180)
-		(fields_autoplaced yes)
 		(effects
 			(font
@@
 		(shape input)
 		(at 53.34 81.28 180)
-		(fields_autoplaced yes)
 		(effects
 			(font
@@
 		(shape output)
 		(at 53.34 83.82 180)
-		(fields_autoplaced yes)
 		(effects
 			(font
@@
 			)
 		)
-		(property "Footprint" "Resistor_SMD:R_0603_1608Metric"
+		(property "Footprint" "Resistor_SMD:R_0402_1005Metric"
 			(at 56.388 90.17 90)
 			(effects
